File: pcb/HE Sensor.kicad_sch (KiCad schematic)
At the start: 119 parts, among them U5 ADG732BSUZ-REEL, U6 ADG732BSUZ-REEL, U7 ADG732BSUZ-REEL, U8 ADG732BSUZ-REEL

Commit message: Normalize line endings to LF
Parts:
- U5, U6, U7, U8: LCSC C114845 -> C579103
Connections:
- no-connect marks 41 -> 140

Commit message: adding flash memory to store user config
Parts:
- renumbered C126 to C127, C127 to C128, C128 to C129, C129 to C130, H4 to H2, H2 to H3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
