File: pcb/LED.kicad_sch (KiCad schematic)
At the start: 198 parts, among them J2 LED_EXP

Commit message: Normalize line endings to LF
Parts:
- R12: LCSC (none) -> C384242
Changed lines of the file:
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@@
+			)
+		)
+		(property "LCSC" "C384242"
+			(at 97.79 33.02 90)
+			(effects
+				(font
+					(size 1.27 1.27)
+				)
+				(hide yes)
 			)
 		)

Commit message: adding flash memory to store user config
Parts:
- renumbered C72 to C100, C73 to C101, C74 to C102, C75 to C103, C76 to C104, C77 to C105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
